File: HC32F460JEUA_robot_controller/HC32F460JEUA_robot_controller.kicad_sch (KiCad schematic)
At the start: 13 parts, among them CN1 XT30PW-M, U1 HC32F460JEUA-QFN48TR, U3 LMR51450SDRRR, U4 CH343P, U5 TJA1051TK-3

Commit message: Update README to reflect project.
Parts:
- added C1, C7: 10u, Capacitor_SMD:C_0603_1608Metric, symbol Library:C0603
- added C2: 100n, Capacitor_SMD:C_0402_1005Metric, symbol Library:C0402
- added D1: PMEG3010ESBYL, Library:SOD993_L1.0-W0.6-LS1.0-RD, symbol Library:PMEG3010ESBYL
Connections:
- net GND: now also U3.13 (EP), U3.6 (RT)
- net +5V: no longer names the net of USB1.A4B9 (VBUS)
- net +5V: now also D1.2
- new net +5V_USB: D1.1
Other:
- moved on the sheet: C3, C4, C5, C6, R1, R2, U3, U4, USB1

Commit message: fix pcb
Parts:
- added C10, C8, C9: 100n, Library:C_0402_1005Metric, symbol Library:C0402
- added C11: 33p, Library:C_0402_1005Metric, symbol Library:C0402
- added C12, C13, C14, C15: 10u, Library:C_0603_1608Metric, symbol Library:C0603
- added CN2: XT30PW-M, Library:AMASS_XT30PW-M_1x02_P2.50mm_Horizontal, symbol Library:XT30PW-M
- added F1: ASMD2920-700-30V, Library:F2920, symbol Library:ASMD2920-700-30V
- added L1: L0630, Library:L_Changjiang_FXL0630, symbol Library:L0630
- added Q1: BSZ088N03MS G, Library:PG-TSDSON-8_L3.3-W3.3-P0.65-BL, symbol Library:BSZ088N03MS G
- added R5: 0, Library:R_0402_1005Metric, symbol Library:R0402
- added R6: 2k, Library:R_0402_1005Metric, symbol Library:R0402
- added R7: 28k, Library:R_0402_1005Metric, symbol Library:R0402
- added R8: 1k, Library:R_0402_1005Metric, symbol Library:R0402
- added U2: TPS54335ADRCR, Library:VSON-10_L3.0-W3.0-P0.50-TL-EP, symbol Library:TPS54335ADRCR
- C1, C7: footprint Capacitor_SMD:C_0603_1608Metric -> Library:C_0603_1608Metric
- C2, C3, C4, C5, C6: footprint Capacitor_SMD:C_0402_1005Metric -> Library:C_0402_1005Metric
- R1, R2, R3: footprint Resistor_SMD:R_0402_1005Metric -> Library:R_0402_1005Metric
Connections:
- net +5V_USB is gone; now on net +5V: D1.1
- net +3.3V: now also U5.5 (VIO), C9.1
- net GND: now also C1.2, C2.2, C7.2, U3.8 (AGND), U5.2 (GND), U5.8 (S), U5.9 (GND), C12.1, C13.1, C14.2, C15.2, C8.2, C9.2, CN2.3, CN2.4, R5.2, R6.2; no longer U3.6 (RT)
- net PGND: now also Q1.1 (S), Q1.2 (S), Q1.3 (S), R5.1
- net +24V: now reaches C7.1
- net +24V: now also C1.1, C2.1, U3.10 (VIN), U3.11 (VIN), U3.12 (VIN), U3.9 (EN)
- net at U3.1 (SW), U3.2 (SW), U3.3 (SW): now also C10.2, L1.2
- net at U3.4 (BOOT): now also C10.1
- net at U3.7 (FB): now also C11.2, R6.1, R7.2
- net +5V: now reaches U5.3 (VCC)
- net +5V: now also C8.1
- net at R3.2, U5.6 (CANL): now also CN2.1 (-)
- net at R3.1, U5.7 (CANH): now also CN2.2 (+)
- net +24V_VCC_IN: no longer names the net of CN1.2 (+)
- net +24V_VCC_IN: now also F1.1
- net CH343_RTS: no longer names the net of U4.13 (~{RTS})
- new net: C11.1, R8.1
- new net: U2.3 (GND), U2.4 (GND), U2.5 (GND)
- new net: Q1.5 (D), Q1.6 (D), Q1.7 (D), Q1.8 (D), Q1.9 (D)
- new net +12V: C12.2, C13.2, C14.1, C15.1, L1.1, R7.1, R8.2
- no-connect marks 8 -> 11
Other:
- note added: "24V_IN->防过流->防反接->防过压"
- note added: "USB_UART"
- note removed: "24V_IN"
- moved on the sheet: C1, C2, C7, CN1, U1, U3
